Commit message: imu urdf 추가 및 encoder 토픽명 변경

File: grandslam_description/urdf/grandslam.xacro (robot description, xacro)
@@ -209,4 +209,12 @@
   <origin xyz="0.18 0 0" rpy="0 0 0"/>
 </joint>
+<!--imu-->
+<link name="imu">
+</link>
+<joint name="imu_joint" type="fixed">
+  <parent link="base_link"/>
+  <child link ="imu"/>
+  <origin xyz="-0.2 0 0" rpy="0 0 0"/>
+</joint>
   <!-- 바퀴 4개 -->
   <xacro:wheel name="wheel_fl" xyz=" 0.18  0.14 0.0"/>

Commit message: Modified node and frame for ekf global

File: grandslam_description/urdf/grandslam.xacro (robot description, xacro)
@@ -217,4 +217,19 @@
   <origin xyz="-0.2 0 0" rpy="0 0 0"/>
 </joint>
+<!-- GPS -->
+<link name="gps">
+  <visual>
+    <origin xyz="0 0 0" rpy="0 0 0"/>
+    <geometry>
+      <sphere radius="0.03"/> <!-- GPS 안테나처럼 작은 구 모양 -->
+    </geometry>
+    <material name="orange"/> <!-- 눈에 띄게 오렌지색 -->
+  </visual>
+</link>
+<joint name="gps_joint" type="fixed">
+  <parent link="base_link"/>
+  <child link="gps"/>
+  <origin xyz="0 0 1" rpy="0 0 0"/> <!-- 차체 위쪽, 살짝 앞쪽 -->
+</joint>
   <!-- 바퀴 4개 -->
   <xacro:wheel name="wheel_fl" xyz=" 0.18  0.14 0.0"/>

Commit message: 동적과 횡단보도 서버 업데이트

File: grandslam_description/urdf/grandslam.xacro (robot description, xacro)
@@ -83,10 +83,25 @@
   <origin xyz="0.25 0 0.075" rpy="0 0 0"/>
 </joint>
-<!-- 2D Lidar -->
+<!-- 라이다 받침 프로파일 직육면체 -->
+<link name="lidar_horizontal">
+  <visual>
+    <origin xyz="0 0 0.06" rpy="0 1.5708 0"/>
+    <geometry>
+      <cylinder length="0.16" radius="0.01"/>
+    </geometry>
+    <material name="black"/>
+  </visual>
+</link>
+<joint name="lidar_horizontal_joint" type="fixed">
+  <parent link="front_bumper"/>
+  <child link="lidar_horizontal"/>
+  <origin xyz="0 0 0.04" rpy="0 0 0"/>
+</joint>
+<!-- 2D Lidar(노랑) -->
 <link name="sensor_tip">
   <visual>
-    <origin xyz="0 0 0.175" rpy="0 0 0"/>
-    <geometry>
-      <cylinder radius="0.02" length="0.05"/>
+    <origin xyz="0.06 0 -0.02" rpy="0 0 0"/>
+    <geometry>
+      <cylinder radius="0.02" length="0.02"/>
     </geometry>
     <material name="yellow"/>
@@ -94,7 +109,14 @@
 </link>
 <joint name="sensor_tip_joint" type="fixed">
-  <parent link="sensor_box"/>
+	<parent link="lidar_horizontal"/>
   <child link="sensor_tip"/>
   <origin xyz="0 0 0.1" rpy="0 0 0"/>
+</joint>
+<!-- Laser frame for Lidar -->
+<link name="laser"/>
+<joint name="laser_joint" type="fixed">
+	<parent link="base_link"/>
+	<child link="laser"/>
+	<origin xyz="1.0 0 0" rpy="0 0 3.14"/>
 </joint>
   <!--  뒷 상자 박스 -->
